File: Clock_design/Clock_design.kicad_pcb (KiCad board)
At the start: 2 copper layers, 118 x 118 mm, 40 parts, among them J1 Conn_02x03_Odd_Even, J2 Power_inlet_vertical, J3 Conn_01x06, Q1 NPN_2N3904_SOT23, SW1 Omron_B3F_SPST, SW2 Omron_B3F_SPST, SW3 Omron_B3F_SPST, SW4 Omron_B3F_SPST, U1 ATmega328-PU, U2 DS1307_DIP-8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

Commit message: Routing done
Parts:
- moved R10 5.92 mm to (137.0, 130.0), turned to -90 degrees
- moved R9 5.81 mm to (177.5, 129.7), turned to -90 degrees
- moved R8 1.20 mm to (157.5, 129.7), turned to -90 degrees
- turned C6 to -90 degrees
Connections:
- DS1 pad 10: NOT CONNECTED -> unconnected-(DS1-Pad10)
- DS1 pad 11: PIN 10 -> D4
- DS1 pad 12: PIN 11 -> D5
- DS1 pad 13: PIN 12 -> D6
- DS1 pad 14: PIN 13 -> D7
- DS1 pad 4: PIN 4 -> RS
- DS1 pad 6: PIN 6 -> E
- DS1 pad 7: NOT CONNECTED -> unconnected-(DS1-Pad7)
- DS1 pad 8: NOT CONNECTED -> unconnected-(DS1-Pad8)
- DS1 pad 9: NOT CONNECTED -> unconnected-(DS1-Pad9)
- R11 pad 1: RXD -> TXD
- R12 pad 1: TXD -> RXD
- RV1 pad 1: unconnected-(RV1-Pad1) -> GND
- RV1 pad 3: unconnected-(RV1-Pad3) -> VCC
- U1 pad 11: LCD_DATA_1 -> D4
- U1 pad 12: LCD_DATA_2 -> D5
- U1 pad 13: LCD_DATA_3 -> D6
- U1 pad 14: LCD_DATA_4 -> D7
- U1 pad 2: unconnected-(U1-Pad2) -> RXD
- U1 pad 24: BUTTON_DWN -> BUTTON_SEL
- U1 pad 25: BUTTON_SEL -> BUTTON_DWN
- U1 pad 3: unconnected-(U1-Pad3) -> TXD
- U1 pad 4: unconnected-(U1-Pad4) -> RS
- U1 pad 5: unconnected-(U1-Pad5) -> E
Routing:
- net BUTTON_SEL: track 0.00 -> 107.0 mm, vias 0 -> 3
- net BUTTON_DWN: track 0.00 -> 85.5 mm, vias 0 -> 1
- net BUTTON_UP: track 0.00 -> 81.6 mm, vias 0 -> 1
- net BUZZER: track 0.00 -> 59.6 mm, vias 0 -> 2
- net RESET: track 0.00 -> 51.1 mm, vias 0 -> 1
- net Net-(DS1-Pad3): track 0.00 -> 43.9 mm
- net RS: track 0.00 -> 40.0 mm, vias 0 -> 2
- net GND: track 0.00 -> 38.3 mm, vias 0 -> 17
- net E: track 0.00 -> 35.5 mm, vias 0 -> 2
- net Net-(BT1-Pad1): track 0.00 -> 33.6 mm
- net SCL: track 0.00 -> 22.3 mm
- net D5: track 0.00 -> 21.5 mm
- net D4: track 0.00 -> 21.5 mm
- net SDA: track 0.00 -> 21.2 mm
- net D7: track 0.00 -> 21.1 mm
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- added copper zone on B.Cu, net GND
- added copper zone on F.Cu, net VCC

Commit message: Routing done Update 2
Parts:
- added D1: LED_0805, footprints:LED_0805_2012Metric, F.Cu at (160.5, 52.5)
- added R13: R_0805_2.2K, footprints:R_0805_2012Metric, F.Cu at (166.5, 56.0)
- C5: value C_0805_0.1uf -> C_0805_1uf
- R5: value R_0805_10K -> R_0805_1K
- moved C5 10.7 mm to (158.3, 126.5)
- moved R5 3.69 mm to (194.7, 101.0)
Routing:
- net Net-(C5-Pad1): track 14.3 -> 25.7 mm
- net LED_SCK: track 8.05 -> 18.9 mm
- net GND: track 38.3 -> 45.8 mm, vias 17 -> 18
- net Net-(D1-Pad1): track 0.00 -> 6.16 mm
- net Net-(Q1-Pad1): track 5.82 -> 9.64 mm
- net BUZZER: track 59.6 -> 62.1 mm

Commit message: Routing Update 3
Parts:
- R7: value R_0805_10K -> R_0805_100K
- moved C5 10.7 mm to (164.2, 135.5)
Connections:
- R7 pad 1: LIGHT_SENSOR -> GND
- R7 pad 2: GND -> LIGHT_SENSOR
Routing:
- net Net-(C5-Pad1): track 25.7 -> 13.8 mm
- net GND: track 45.8 -> 36.4 mm
- net LIGHT_SENSOR: track 13.9 -> 10.8 mm
- net BUZZER: track 62.1 -> 59.7 mm
Changed lines of the file:
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@@
     )
     (pad_to_mask_clearance 0)
+    (aux_axis_origin 91 159)
     (pcbplotparams
       (layerselection 0x00010fc_ffffffff)
@@
     (property "Tolerance" "N/A")
     (attr smd)
-    (fp_text reference "R13" (at 0 -1.65 90) (layer "F.SilkS")
+    (fp_text reference "R13" (at 0 2 90) (layer "F.SilkS")
       (effects (font (size 1 1) (thickness 0.15)))
     )
@@
   )
   (footprint "footprints:C_0805_2012Metric" (layer "F.Cu")
-    (at 158.35 126.5)
+    (at 164.15 135.5)
     (descr "Capacitor SMD 0805 (2012 Metric), square (rectangular) end terminal, IPC_7351 nominal, (Body size source: http://www.tortai-tech.com/upload/download/2011102023233369053.pdf), generated with kicad-footprint-generator")
     (tags "capacitor")
@@
     (descr "Resistor SMD 0805 (2012 Metric), square (rectangular) end terminal, IPC_7351 nominal, (Body size source: http://www.tortai-tech.com/upload/download/2011102023233369053.pdf), generated with kicad-footprint-generator")
     (tags "resistor")
-    (property "Digikey PN" "311-10.0KCRCT-ND")
+    (property "Digikey PN" "311-100KCRCT-ND")
     (property "MFG" "Yageo")
-    (property "MPN" "RC0805FR-0710KL")
+    (property "MPN" "RC0805FR-07100KL")
     (property "Mouser PN" "N/A")
     (property "Power" "N/A")
@@
       (effects (font (size 1 1) (thickness 0.15)))
     )
-    (fp_text value "R_0805_10K" (at 0 1.65) (layer "F.Fab")
+    (fp_text value "R_0805_100K" (at 0 1.65) (layer "F.Fab")
       (effects (font (size 1 1) (thickness 0.15)))
     )
@@
     (fp_line (start -1 0.6) (end -1 -0.6) (layer "F.Fab") (width 0.1))
     (pad "1" smd rect locked (at -0.85 0) (size 1.15 1.4) (layers "F.Cu" "F.Paste" "F.Mask")
+      (net 2 "GND") (pintype "passive"))
+    (pad "2" smd rect locked (at 0.85 0) (size 1.15 1.4) (layers "F.Cu" "F.Paste" "F.Mask")
       (net 21 "LIGHT_SENSOR") (pintype "passive"))
-    (pad "2" smd rect locked (at 0.85 0) (size 1.15 1.4) (layers "F.Cu" "F.Paste" "F.Mask")
-      (net 2 "GND") (pintype "passive"))
     (model "${HPS3DMOD}/R_0805_2012Metric.wrl"
       (offset (xyz 0 0 0))
@@
     (property "Sheetname" "")
     (attr smd)
-    (fp_text reference "D1" (at 0 -1.65) (layer "F.SilkS")
+    (fp_text reference "D1" (at 2.5 0) (layer "F.SilkS")
       (effects (font (size 1 1) (thickness 0.15)))
     )
@@
     (fp_arc (start -0.29972 8.49884) (mid -0.153162 8.145018) (end 0.20066 7.99846) (layer "F.SilkS") (width 0.12))
     (fp_arc (start 0.20066 22.9997) (mid -0.153162 22.853142) (end -0.29972 22.49932) (layer "F.SilkS") (width 0.12))
-    (fp_arc (start 64.20104 22.49932) (mid 64.054479 22.85315) (end 63.70066 22.9997) (layer "F.SilkS") (width 0.12))
+    (fp_arc (start 64.20104 22.49932) (mid 64.054473 22.853115) (end 63.70066 22.9997) (layer "F.SilkS") (width 0.12))
     (fp_line (start -8.25 33.75) (end 72.25 33.75) (layer "F.CrtYd") (width 0.05))
     (fp_line (start -8.25 -2.75) (end -8.25 33.75) (layer "F.CrtYd") (width 0.05))
@@
   (segment (start 142 55.25) (end 142 56.5) (width 0.25) (layer "F.Cu") (net 2))
   (segment (start 134 125.75) (end 134 123.5) (width 0.25) (layer "F.Cu") (net 2))
-  (segment (start 149.24 63.68) (end 149.24 61.39) (width 0.25) (layer "F.Cu") (net 2))
   (segment (start 154 125.75) (end 154 123.5) (width 0.25) (layer "F.Cu") (net 2))
   (segment (start 166 125.75) (end 166 123.5) (width 0.25) (layer "F.Cu") (net 2))
   (segment (start 167.5 80.5) (end 167.5 82) (width 0.25) (layer "F.Cu") (net 2))
-  (segment (start 149.24 61.39) (end 148.35 60.5) (width 0.25) (layer "F.Cu") (net 2))
   (segment (start 126 125.75) (end 126 123.5) (width 0.25) (layer "F.Cu") (net 2))
-  (segment (start 154.274511 125.475489) (end 158.399511 125.475489) (width 0.25) (layer "F.Cu") (net 2))
   (segment (start 166.5 56.85) (end 166.5 58.5) (width 0.25) (layer "F.Cu") (net 2))
   (segment (start 146 125.75) (end 146 123.5) (width 0.25) (layer "F.Cu") (net 2))
@@
   (segment (start 158.85 80) (end 158.85 81.35) (width 0.25) (layer "F.Cu") (net 2))
   (segment (start 191.5 110.95) (end 191.5 112.5) (width 0.25) (layer "F.Cu") (net 2))
-  (segment (start 159.2 126.275978) (end 159.2 126.5) (width 0.25) (layer "F.Cu") (net 2))
-  (segment (start 154 125.75) (end 154.274511 125.475489) (width 0.25) (layer "F.Cu") (net 2))
   (segment (start 157.65 147.65) (end 158 148) (width 0.25) (layer "F.Cu") (net 2))
   (segment (start 169.825 136.675) (end 169.825 140.325) (width 1) (layer "F.Cu") (net 2))
   (segment (start 165 135.5) (end 166.5 135.5) (width 1) (layer "F.Cu") (net 2))
-  (segment (start 158.399511 125.475489) (end 159.2 126.275978) (width 0.25) (layer "F.Cu") (net 2))
   (segment (start 157.65 146.35) (end 157.65 147.65) (width 0.5) (layer "F.Cu") (net 2))
   (segment (start 168.5 135.5) (end 169.825 135.5) (width 1) (layer "F.Cu") (net 2))
@@
   (segment (start 161.56 76) (end 156.86 71.3) (width 0.25) (layer "F.Cu") (net 7))
   (segment (start 155.085 138.745) (end 153.5 137.16) (width 1) (layer "F.Cu") (net 8))
-  (segment (start 163 138.22) (end 163 135.8) (width 1) (layer "F.Cu") (net 8))
-  (segment (start 157.5 126.625) (end 163.3 132.425) (width 0.25) (layer "F.Cu") (net 8))
-  (segment (start 163 135.8) (end 163.3 135.5) (width 1) (layer "F.Cu") (net 8))
+  (segment (start 163 135.8) (end 163 136.5) (width 0.25) (layer "F.Cu") (net 8))
   (segment (start 163.525 138.745) (end 155.085 138.745) (width 1) (layer "F.Cu") (net 8))
   (segment (start 163.525 138.745) (end 163 138.22) (width 1) (layer "F.Cu") (net 8))
-  (segment (start 157.5 126.5) (end 157.5 126.625) (width 0.25) (layer "F.Cu") (net 8))
-  (segment (start 163.3 132.425) (end 163.3 135.5) (width 0.25) (layer "F.Cu") (net 8))
+  (segment (start 163 138.22) (end 163 136.5) (width 1) (layer "F.Cu") (net 8))
   (segment (start 160.880489 55.550489) (end 162.055 56.725) (width 0.25) (layer "F.Cu") (net 9))
   (segment (start 134 58) (end 134 59.75) (width 0.25) (layer "F.Cu") (net 9))
@@
   (segment (start 126.9 73.32) (end 136.54 63.68) (width 0.25) (layer "F.Cu") (net 19))
   (segment (start 124.32 73.32) (end 124.32 78.32) (width 0.25) (layer "F.Cu") (net 19))
-  (segment (start 191.65 101.65) (end 191.65 101.85) (width 0.25) (layer "F.Cu") (net 20))
   (segment (start 192.5 101) (end 191.65 101.85) (width 0.25) (layer "F.Cu") (net 20))
   (segment (start 193.8 101) (end 192.5 101) (width 0.25) (layer "F.Cu") (net 20))
   (segment (start 167.02 63.68) (end 181.82 63.68) (width 0.25) (layer "F.Cu") (net 20))
   (segment (start 181.82 63.68) (end 182 63.5) (width 0.25) (layer "F.Cu") (net 20))
-  (segment (start 191.65 101.85) (end 191.65 104) (width 0.25) (layer "F.Cu") (net 20))
   (segment (start 191 101) (end 191.65 101.65) (width 0.25) (layer "F.Cu") (net 20))
   (via (at 182 63.5) (size 0.8) (drill 0.4) (layers "F.Cu" "B.Cu") (net 20))
@@
   (segment (start 182 63.5) (end 182 92) (width 0.25) (layer "B.Cu") (net 20))
   (segment (start 182 92) (end 191 101) (width 0.25) (layer "B.Cu") (net 20))
-  (segment (start 146.7 63.68) (end 146.7 60.55) (width 0.25) (layer "F.Cu") (net 21))
   (segment (start 148.2 62.18) (end 146.7 63.68) (width 0.25) (layer "B.Cu") (net 21))
   (segment (start 148.2 53.5) (end 148.2 62.18) (width 0.25) (layer "B.Cu") (net 21))

Commit message: Routing Update 4
Routing:
- net LIGHT_SENSOR: track 10.8 -> 14.7 mm
- net GND: track 36.4 -> 37.9 mm, vias 18 -> 19
Changed lines of the file:
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@@
     (fp_arc (start -0.29972 8.49884) (mid -0.153162 8.145018) (end 0.20066 7.99846) (layer "F.SilkS") (width 0.12))
     (fp_arc (start 0.20066 22.9997) (mid -0.153162 22.853142) (end -0.29972 22.49932) (layer "F.SilkS") (width 0.12))
-    (fp_arc (start 64.20104 22.49932) (mid 64.054473 22.853115) (end 63.70066 22.9997) (layer "F.SilkS") (width 0.12))
+    (fp_arc (start 64.20104 22.49932) (mid 64.054479 22.85315) (end 63.70066 22.9997) (layer "F.SilkS") (width 0.12))
     (fp_line (start -8.25 33.75) (end 72.25 33.75) (layer "F.CrtYd") (width 0.05))
     (fp_line (start -8.25 -2.75) (end -8.25 33.75) (layer "F.CrtYd") (width 0.05))
@@
   (segment (start 142 55.25) (end 142 56.5) (width 0.25) (layer "F.Cu") (net 2))
   (segment (start 134 125.75) (end 134 123.5) (width 0.25) (layer "F.Cu") (net 2))
+  (segment (start 146.65 60.5) (end 146.65 61.85) (width 0.25) (layer "F.Cu") (net 2))
   (segment (start 154 125.75) (end 154 123.5) (width 0.25) (layer "F.Cu") (net 2))
   (segment (start 166 125.75) (end 166 123.5) (width 0.25) (layer "F.Cu") (net 2))
@@
   (segment (start 134 55.25) (end 134 56.5) (width 0.25) (layer "F.Cu") (net 2))
   (segment (start 152 59.8) (end 152 58.5) (width 0.25) (layer "F.Cu") (net 2))
+  (segment (start 146.65 61.85) (end 146.5 62) (width 0.25) (layer "F.Cu") (net 2))
   (segment (start 166.5 135.5) (end 168.5 135.5) (width 1) (layer "F.Cu") (net 2))
   (segment (start 153 74.5) (end 153 75.85) (width 0.25) (layer "F.Cu") (net 2))
@@
   (via (at 159 81.5) (size 0.8) (drill 0.4) (layers "F.Cu" "B.Cu") (net 2))
   (via (at 166.5 135.5) (size 0.8) (drill 0.4) (layers "F.Cu" "B.Cu") (net 2))
+  (via (at 146.5 62) (size 0.8) (drill 0.4) (layers "F.Cu" "B.Cu") (net 2))
   (via (at 134 56.5) (size 0.8) (drill 0.4) (layers "F.Cu" "B.Cu") (net 2))
   (via (at 126 123.5) (size 0.8) (drill 0.4) (layers "F.Cu" "B.Cu") (net 2))
@@
   (segment (start 182 63.5) (end 182 92) (width 0.25) (layer "B.Cu") (net 20))
   (segment (start 182 92) (end 191 101) (width 0.25) (layer "B.Cu") (net 20))
+  (segment (start 148.35 60.5) (end 148.35 62.03) (width 0.25) (layer "F.Cu") (net 21))
+  (segment (start 148.35 62.03) (end 146.7 63.68) (width 0.25) (layer "F.Cu") (net 21))
   (segment (start 148.2 62.18) (end 146.7 63.68) (width 0.25) (layer "B.Cu") (net 21))
   (segment (start 148.2 53.5) (end 148.2 62.18) (width 0.25) (layer "B.Cu") (net 21))

Commit message: Final Gerber Out
Parts:
- added G***: LOGO, LOGO, B.Cu at (179.1, 99.9)
- added G***: LOGO, LOGO, B.Cu at (136.7, 103.7)
Other:
- board text added: "Desvaun's HPS 2022 Clock"
