File: Clock_design/Clock_design.kicad_sch (KiCad schematic)
At the start: 40 parts, among them J1 Conn_02x03_Odd_Even, J2 Power_inlet_vertical, J3 Conn_01x06, Q1 NPN_2N3904_SOT23, SW1 Omron_B3F_SPST, SW2 Omron_B3F_SPST, SW3 Omron_B3F_SPST, SW4 Omron_B3F_SPST, U1 ATmega328-PU, U2 DS1307_DIP-8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

Commit message: Routing done
Connections:
- net PIN 10 is gone; now on net D4: DS1.11 (D4)
- net PIN 11 is gone; now on net D5: DS1.12 (D5)
- net PIN 12 is gone; now on net D6: DS1.13 (D6)
- net PIN 13 is gone; now on net D7: DS1.14 (D7)
- net PIN 4 is gone; now on net RS: DS1.4 (RS)
- net PIN 6 is gone; now on net E: DS1.6 (E)
- net BUTTON_DWN: now also U1.25 (ADC2/PC2); no longer U1.24 (ADC1/PC1)
- net BUTTON_SEL: now also U1.24 (ADC1/PC1); no longer U1.25 (ADC2/PC2)
- net GND: now also RV1.1
- net RXD: now also R12.1, U1.2 (RXD/PD0); no longer R11.1
- net TXD: now also R11.1, U1.3 (TXD/PD1); no longer R12.1
- net VCC: now also RV1.3
- net RS: now reaches U1.4 (INT0/PD2)
- net E: now reaches U1.5 (INT1/PD3)
- net LCD_DATA_1 renamed D4
- net LCD_DATA_2 renamed D5
- net LCD_DATA_3 renamed D6
- net LCD_DATA_4 renamed D7
- removed net NOT CONNECTED: DS1.10 (D3), DS1.7 (D0), DS1.8 (D1), DS1.9 (D2)
- no-connect marks 2 -> 9
Other:
- moved on the sheet: DS1, RV1

Commit message: Routing done Update 2
Parts:
- removed C5: C_0805_0.1uf, footprints:C_0805_2012Metric, symbol HPS:C_0805_0.1uf
- removed R5: R_0805_10K, footprints:R_0805_2012Metric, symbol HPS:R_0805_10K
- added C5: C_0805_1uf, footprints:C_0805_2012Metric, symbol HPS:C_0805_1uf
- added D1: LED_0805, footprints:LED_0805_2012Metric, symbol HPS:LED_0805
- added R13: R_0805_2.2K, footprints:R_0805_2012Metric, symbol HPS:R_0805_2.2K
- added R5: R_0805_1K, footprints:R_0805_2012Metric, symbol HPS:R_0805_1K
Connections:
- net BUZZER: now also R5.1
- net GND: now also C5.2, R13.1
- net LED_SCK: now also D1.2 (A)
- net at Q1.1 (B): now also R5.2
- net at J2.1 (POLE), U3.1 (IN): now also C5.1
- new net: D1.1 (K), R13.2
Other:
- note added: "BUTTONS"
- note added: "BUZZER"
- note added: "ICSP"
- note added: "LCD"
- note added: "LED"
- note added: "LIGHT SENSOR"
- note added: "MCU"
- note added: "POWER SUPPLY"
- note added: "REAL TIME CLOCK"
- note added: "SERIAL"

Commit message: Routing Update 3
Parts:
- removed R7: R_0805_10K, footprints:R_0805_2012Metric, symbol HPS:R_0805_10K
- added R7: R_0805_100K, footprints:R_0805_2012Metric, symbol HPS:R_0805_100K
Connections:
- net GND: now also R7.1
- net LIGHT_SENSOR: now also R7.2
Changed lines of the file:
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@@
+    (pin "2")
+  )
+  (symbol (lib_id "HPS:R_0805_100K") (at 73.66 240.03 180) (unit 1)
+    (in_bom yes) (on_board yes) (fields_autoplaced)
+    (property "Reference" "R7" (id 0) (at 76.2 238.7599 0)
+      (effects (font (size 1.27 1.27)) (justify right))
+    )
+    (property "Value" "R_0805_100K" (id 1) (at 76.2 241.2999 0)
+      (effects (font (size 1.27 1.27)) (justify right))
+    )
+    (property "Footprint" "footprints:R_0805_2012Metric" (id 2) (at 73.66 223.52 0)
+      (effects (font (size 1.27 1.27)) hide)
+    )
+    (property "Datasheet" "https://www.digikey.com/en/products/detail/yageo/RC0805FR-07100KL/727544" (id 3) (at 76.2 240.03 0)
+      (effects (font (size 1.27 1.27)) hide)
+    )
+    (property "MFG" "Yageo" (id 4) (at 73.66 228.6 0)
+      (effects (font (size 1.27 1.27)) hide)
+    )
+    (property "MPN" "RC0805FR-07100KL" (id 5) (at 73.66 226.06 0)
+      (effects (font (size 1.27 1.27)) hide)
+    )
+    (property "Digikey PN" "311-100KCRCT-ND" (id 6) (at 73.66 220.98 0)
+      (effects (font (size 1.27 1.27)) hide)
+    )
+    (property "Mouser PN" "N/A" (id 7) (at 73.66 218.44 0)
+      (effects (font (size 1.27 1.27)) hide)
+    )
+    (property "Power" "N/A" (id 8) (at 73.66 215.9 0)
+      (effects (font (size 1.27 1.27)) hide)
+    )
+    (property "Tolerance" "N/A" (id 9) (at 73.66 213.36 0)
+      (effects (font (size 1.27 1.27)) hide)
+    )
+    (pin "1")
     (pin "2")
   )
@@
     )
     (property "MPN" "RC0805FR-071KL" (id 9) (at 91.44 173.99 0)
-      (effects (font (size 1.27 1.27)) hide)
-    )
-    (pin "1")
-    (pin "2")
-  )
-  (symbol (lib_id "HPS:R_0805_10K") (at 73.66 240.03 0) (unit 1)
-    (in_bom yes) (on_board yes) (fields_autoplaced)
-    (property "Reference" "R7" (id 0) (at 76.2 238.7599 0)
-      (effects (font (size 1.27 1.27)) (justify left))
-    )
-    (property "Value" "R_0805_10K" (id 1) (at 76.2 241.2999 0)
-      (effects (font (size 1.27 1.27)) (justify left))
-    )
-    (property "Footprint" "footprints:R_0805_2012Metric" (id 2) (at 73.66 256.54 0)
-      (effects (font (size 1.27 1.27)) hide)
-    )
-    (property "Datasheet" "https://www.digikey.com/en/products/detail/yageo/RC0805FR-0710KL/727535" (id 3) (at 71.12 240.03 0)
-      (effects (font (size 1.27 1.27)) hide)
-    )
-    (property "MFG" "Yageo" (id 4) (at 73.66 251.46 0)
-      (effects (font (size 1.27 1.27)) hide)
-    )
-    (property "MPN" "RC0805FR-0710KL" (id 5) (at 73.66 254 0)
-      (effects (font (size 1.27 1.27)) hide)
-    )
-    (property "Digikey PN" "311-10.0KCRCT-ND" (id 6) (at 73.66 259.08 0)
-      (effects (font (size 1.27 1.27)) hide)
-    )
-    (property "Mouser PN" "N/A" (id 7) (at 73.66 261.62 0)
-      (effects (font (size 1.27 1.27)) hide)
-    )
-    (property "Power" "N/A" (id 8) (at 73.66 264.16 0)
-      (effects (font (size 1.27 1.27)) hide)
-    )
-    (property "Tolerance" "N/A" (id 9) (at 73.66 266.7 0)
       (effects (font (size 1.27 1.27)) hide)
     )
@@
       (reference "R6") (unit 1) (value "PhotoconductivePhotocell") (footprint "footprints:R_LDR_4.9x4.2mm_P2.54mm_Vertical")
     )
-    (path "/5e6eada3-2f11-4981-9bd2-69d6f6375c6c"
-      (reference "R7") (unit 1) (value "R_0805_10K") (footprint "footprints:R_0805_2012Metric")
+    (path "/0bf32004-4913-4f13-884f-3ad0e36183c5"
+      (reference "R7") (unit 1) (value "R_0805_100K") (footprint "footprints:R_0805_2012Metric")
     )
     (path "/806ac943-a098-4def-bb09-8cc68e6a3938"

Commit message: Final Gerber Out
Changed lines of the file:
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@@
     (pin "2")
+  )
+  (symbol (lib_id "HPS:HPS_Logo") (at 323.85 36.83 0) (unit 1)
+    (in_bom yes) (on_board yes) (fields_autoplaced)
+    (property "Reference" "#G1" (id 0) (at 323.85 29.9604 0)
+      (effects (font (size 1.27 1.27)) hide)
+    )
+    (property "Value" "HPS_Logo" (id 1) (at 323.85 43.6996 0)
+      (effects (font (size 1.27 1.27)) hide)
+    )
+    (property "Footprint" "" (id 2) (at 323.85 36.83 0)
+      (effects (font (size 1.27 1.27)) hide)
+    )
+    (property "Datasheet" "" (id 3) (at 323.85 36.83 0)
+      (effects (font (size 1.27 1.27)) hide)
+    )
   )
   (symbol (lib_id "HPS:LED_0805") (at 372.11 36.83 90) (unit 1)
@@
       (reference "#FLG03") (unit 1) (value "PWR_FLAG") (footprint "")
     )
+    (path "/6daec851-6a2e-4cad-ae70-3c82216bdeb2"
+      (reference "#G1") (unit 1) (value "HPS_Logo") (footprint "")
+    )
     (path "/57abbc56-26a5-4e47-a4e9-c95c2fe916ed"
